File: 16A.kicad_sch (KiCad schematic)
At the start: 34 parts, among them SW1 SW_DIP_x01, U1 ProMicro

Commit message: Schematics & PCB update
Parts:
- D1, D10, D11, D12, D13, D14, D15, D16, D2, D3, D4, D5, D6, D7, D8, D9: footprint (none) -> Diode_SMD:D_SOD-123
- MX1, MX10, MX11, MX12, MX13, MX14, MX15, MX16, MX2, MX3, MX4, MX5, MX6, MX7, MX8, MX9: footprint PCM_marbastlib-mx:SW_MX_HS_1u -> marbastlib-mx:SW_MX_HS_1u
- SW1: footprint (none) -> Switches:TACTILE_SWITCH_SMD_6.0X3.5MM
- U1: footprint PCM_marbastlib-xp-promicroish:ProMicro_USBup -> marbastlib-xp-promicroish:ProMicro_USBup
Changed lines of the file:
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@@
       (effects (font (size 1.27 1.27)))
     )
-    (property "Footprint" "PCM_marbastlib-mx:SW_MX_HS_1u" (at 139.7 63.5 0)
+    (property "Footprint" "marbastlib-mx:SW_MX_HS_1u" (at 139.7 63.5 0)
       (effects (font (size 1.27 1.27)) hide)
     )
@@
       (effects (font (size 1.27 1.27)))
     )
-    (property "Footprint" "PCM_marbastlib-mx:SW_MX_HS_1u" (at 127 81.28 0)
+    (property "Footprint" "marbastlib-mx:SW_MX_HS_1u" (at 127 81.28 0)
       (effects (font (size 1.27 1.27)) hide)
     )
@@
       (effects (font (size 1.27 1.27)) (justify right))
     )
-    (property "Footprint" "" (at 167.64 104.14 90)
+    (property "Footprint" "Diode_SMD:D_SOD-123" (at 167.64 104.14 90)
       (effects (font (size 1.27 1.27)) hide)
     )
@@
       (effects (font (size 1.27 1.27)))
     )
-    (property "Footprint" "PCM_marbastlib-mx:SW_MX_HS_1u" (at 165.1 99.06 0)
+    (property "Footprint" "marbastlib-mx:SW_MX_HS_1u" (at 165.1 99.06 0)
       (effects (font (size 1.27 1.27)) hide)
     )
@@
       (effects (font (size 1.27 1.27)) (justify right))
     )
-    (property "Footprint" "" (at 154.94 86.36 90)
+    (property "Footprint" "Diode_SMD:D_SOD-123" (at 154.94 86.36 90)
       (effects (font (size 1.27 1.27)) hide)
     )
@@
       (effects (font (size 1.27 1.27)))
     )
-    (property "Footprint" "PCM_marbastlib-mx:SW_MX_HS_1u" (at 152.4 99.06 0)
+    (property "Footprint" "marbastlib-mx:SW_MX_HS_1u" (at 152.4 99.06 0)
       (effects (font (size 1.27 1.27)) hide)
     )
@@
       (effects (font (size 1.27 1.27)) (justify right))
     )
-    (property "Footprint" "" (at 129.54 68.58 90)
+    (property "Footprint" "Diode_SMD:D_SOD-123" (at 129.54 68.58 90)
       (effects (font (size 1.27 1.27)) hide)
     )
@@
       (effects (font (size 1.27 1.27)) (justify right))
     )
-    (property "Footprint" "" (at 154.94 68.58 90)
+    (property "Footprint" "Diode_SMD:D_SOD-123" (at 154.94 68.58 90)
       (effects (font (size 1.27 1.27)) hide)
     )
@@
       (effects (font (size 1.27 1.27)))
     )
-    (property "Footprint" "PCM_marbastlib-mx:SW_MX_HS_1u" (at 127 63.5 0)
+    (property "Footprint" "marbastlib-mx:SW_MX_HS_1u" (at 127 63.5 0)
       (effects (font (size 1.27 1.27)) hide)
     )
@@
       (effects (font (size 1.27 1.27)))
     )
-    (property "Footprint" "PCM_marbastlib-mx:SW_MX_HS_1u" (at 139.7 99.06 0)
+    (property "Footprint" "marbastlib-mx:SW_MX_HS_1u" (at 139.7 99.06 0)
       (effects (font (size 1.27 1.27)) hide)
     )
@@
       (effects (font (size 1.27 1.27)))
     )
-    (property "Footprint" "PCM_marbastlib-mx:SW_MX_HS_1u" (at 152.4 116.84 0)
+    (property "Footprint" "marbastlib-mx:SW_MX_HS_1u" (at 152.4 116.84 0)
       (effects (font (size 1.27 1.27)) hide)
     )
@@
       (effects (font (size 1.27 1.27)) (justify right))
     )
-    (property "Footprint" "" (at 154.94 104.14 90)
+    (property "Footprint" "Diode_SMD:D_SOD-123" (at 154.94 104.14 90)
       (effects (font (size 1.27 1.27)) hide)
     )
@@
       (effects (font (size 1.27 1.27)) (justify right))
     )
-    (property "Footprint" "" (at 129.54 121.92 90)
+    (property "Footprint" "Diode_SMD:D_SOD-123" (at 129.54 121.92 90)
       (effects (font (size 1.27 1.27)) hide)
     )
@@
       (effects (font (size 1.27 1.27)) (justify right))
     )
-    (property "Footprint" "" (at 142.24 86.36 90)
+    (property "Footprint" "Diode_SMD:D_SOD-123" (at 142.24 86.36 90)
       (effects (font (size 1.27 1.27)) hide)
     )
@@
       (effects (font (size 1.27 1.27)))
     )
-    (property "Footprint" "PCM_marbastlib-mx:SW_MX_HS_1u" (at 127 99.06 0)
+    (property "Footprint" "marbastlib-mx:SW_MX_HS_1u" (at 127 99.06 0)
       (effects (font (size 1.27 1.27)) hide)
     )
@@
       (effects (font (size 1.27 1.27)) (justify right))
     )
-    (property "Footprint" "" (at 142.24 121.92 90)
+    (property "Footprint" "Diode_SMD:D_SOD-123" (at 142.24 121.92 90)
       (effects (font (size 1.27 1.27)) hide)
     )
@@
       (effects (font (size 1.27 1.27)))
     )
-    (property "Footprint" "PCM_marbastlib-xp-promicroish:ProMicro_USBup" (at 67.31 110.49 0)
+    (property "Footprint" "marbastlib-xp-promicroish:ProMicro_USBup" (at 67.31 110.49 0)
       (effects (font (size 1.27 1.27)) hide)
     )
@@
       (effects (font (size 1.27 1.27)) (justify right))
     )
-    (property "Footprint" "" (at 167.64 121.92 90)
+    (property "Footprint" "Diode_SMD:D_SOD-123" (at 167.64 121.92 90)
       (effects (font (size 1.27 1.27)) hide)
     )
@@
       (effects (font (size 1.27 1.27)) (justify right))
     )
-    (property "Footprint" "" (at 142.24 104.14 90)
+    (property "Footprint" "Diode_SMD:D_SOD-123" (at 142.24 104.14 90)
       (effects (font (size 1.27 1.27)) hide)
     )
@@
       (effects (font (size 1.27 1.27)) (justify right))
     )
-    (property "Footprint" "" (at 167.64 86.36 90)
+    (property "Footprint" "Diode_SMD:D_SOD-123" (at 167.64 86.36 90)
       (effects (font (size 1.27 1.27)) hide)
     )
@@
       (effects (font (size 1.27 1.27)) (justify right))
     )
-    (property "Footprint" "" (at 129.54 104.14 90)
+    (property "Footprint" "Diode_SMD:D_SOD-123" (at 129.54 104.14 90)
       (effects (font (size 1.27 1.27)) hide)
     )
@@
       (effects (font (size 1.27 1.27)) (justify right))
     )
-    (property "Footprint" "" (at 129.54 86.36 90)
+    (property "Footprint" "Diode_SMD:D_SOD-123" (at 129.54 86.36 90)
       (effects (font (size 1.27 1.27)) hide)
     )
@@
       (effects (font (size 1.27 1.27)))
     )
-    (property "Footprint" "PCM_marbastlib-mx:SW_MX_HS_1u" (at 152.4 63.5 0)
+    (property "Footprint" "marbastlib-mx:SW_MX_HS_1u" (at 152.4 63.5 0)
       (effects (font (size 1.27 1.27)) hide)
     )
@@
       (effects (font (size 1.27 1.27)) (justify right))
     )
-    (property "Footprint" "" (at 154.94 121.92 90)
+    (property "Footprint" "Diode_SMD:D_SOD-123" (at 154.94 121.92 90)
       (effects (font (size 1.27 1.27)) hide)
     )
@@
       (effects (font (size 1.27 1.27)))
     )
-    (property "Footprint" "PCM_marbastlib-mx:SW_MX_HS_1u" (at 152.4 81.28 0)
+    (property "Footprint" "marbastlib-mx:SW_MX_HS_1u" (at 152.4 81.28 0)
       (effects (font (size 1.27 1.27)) hide)
     )
@@
       (effects (font (size 1.27 1.27)))
     )
-    (property "Footprint" "" (at 95.25 67.31 0)
+    (property "Footprint" "Switches:TACTILE_SWITCH_SMD_6.0X3.5MM" (at 95.25 67.31 0)
       (effects (font (size 1.27 1.27)) hide)
     )
@@
       (effects (font (size 1.27 1.27)))
     )
-    (property "Footprint" "PCM_marbastlib-mx:SW_MX_HS_1u" (at 139.7 81.28 0)
+    (property "Footprint" "marbastlib-mx:SW_MX_HS_1u" (at 139.7 81.28 0)
       (effects (font (size 1.27 1.27)) hide)
     )
@@
       (effects (font (size 1.27 1.27)) (justify right))
     )
-    (property "Footprint" "" (at 142.24 68.58 90)
+    (property "Footprint" "Diode_SMD:D_SOD-123" (at 142.24 68.58 90)
       (effects (font (size 1.27 1.27)) hide)
     )
@@
       (effects (font (size 1.27 1.27)))
     )
-    (property "Footprint" "PCM_marbastlib-mx:SW_MX_HS_1u" (at 165.1 81.28 0)
+    (property "Footprint" "marbastlib-mx:SW_MX_HS_1u" (at 165.1 81.28 0)
       (effects (font (size 1.27 1.27)) hide)
     )
@@
       (effects (font (size 1.27 1.27)))
     )
-    (property "Footprint" "PCM_marbastlib-mx:SW_MX_HS_1u" (at 127 116.84 0)
+    (property "Footprint" "marbastlib-mx:SW_MX_HS_1u" (at 127 116.84 0)
       (effects (font (size 1.27 1.27)) hide)
     )
@@
       (effects (font (size 1.27 1.27)))
     )
-    (property "Footprint" "PCM_marbastlib-mx:SW_MX_HS_1u" (at 165.1 116.84 0)
+    (property "Footprint" "marbastlib-mx:SW_MX_HS_1u" (at 165.1 116.84 0)
       (effects (font (size 1.27 1.27)) hide)
     )
@@
       (effects (font (size 1.27 1.27)) (justify right))
     )
-    (property "Footprint" "" (at 167.64 68.58 90)
+    (property "Footprint" "Diode_SMD:D_SOD-123" (at 167.64 68.58 90)
       (effects (font (size 1.27 1.27)) hide)
     )
@@
       (effects (font (size 1.27 1.27)))
     )
-    (property "Footprint" "PCM_marbastlib-mx:SW_MX_HS_1u" (at 139.7 116.84 0)
+    (property "Footprint" "marbastlib-mx:SW_MX_HS_1u" (at 139.7 116.84 0)
       (effects (font (size 1.27 1.27)) hide)
     )
@@
       (effects (font (size 1.27 1.27)))
     )
-    (property "Footprint" "PCM_marbastlib-mx:SW_MX_HS_1u" (at 165.1 63.5 0)
-      (effects (font (size 1.27 1.27)) hide)
-    )
+    (property "Footprint" "marbastlib-mx:SW_MX_HS_1u" (at 165.1 63.5 0)
+      (effects (font (size 1.27 1.27)) hide)
+    )
